Commit message: add gripper

File: src/mycobot_description/urdf/mycobot.xacro (robot description, xacro)
@@ -1,188 +1,375 @@
 <?xml version="1.0" ?>
-<robot name="mycobot320" xmlns:xacro="http://www.ros.org/wiki/xacro">
+<robot name="mycobot" xmlns:xacro="http://www.ros.org/wiki/xacro">
 <xacro:include filename="$(find mycobot_description)/urdf/materials.xacro" />
-  <link name="base_link">
-    <inertial>
-      <origin xyz="-1.3994637957346424e-08 0.046320428630226694 0.053625500753973876" rpy="0 0 0"/>
-      <mass value="12.899764355948896"/>
-      <inertia ixx="0.033823" iyy="0.028162" izz="0.035033" ixy="0.0" iyz="-0.000755" ixz="0.0"/>
-    </inertial>
-    <visual>
-      <origin xyz="0 0 0" rpy="0 0 0"/>
-      <geometry>
-        <mesh filename="file://$(find mycobot_description)/meshes/base_link.stl" scale="0.001 0.001 0.001"/>
-      </geometry>
-      <material name="silver"/>
-    </visual>
-    <collision>
-      <origin xyz="0 0 0" rpy="0 0 0"/>
-      <geometry>
-        <mesh filename="file://$(find mycobot_description)/meshes/base_link.stl" scale="0.001 0.001 0.001"/>
-      </geometry>
-    </collision>
-  </link>
-  <link name="link1">
-    <inertial>
-      <origin xyz="0.0068967662247303866 -3.47113377312247e-07 0.055490142550686156" rpy="0 0 0"/>
-      <mass value="3.4735206294395446"/>
-      <inertia ixx="0.004461" iyy="0.004757" izz="0.002424" ixy="0.0" iyz="0.0" ixz="-0.000777"/>
-    </inertial>
-    <visual>
-      <origin xyz="0.0 -0.060072 -0.114761" rpy="0 0 0"/>
-      <geometry>
-        <mesh filename="file://$(find mycobot_description)/meshes/link1.stl" scale="0.001 0.001 0.001"/>
-      </geometry>
-      <material name="silver"/>
-    </visual>
-    <collision>
-      <origin xyz="0.0 -0.060072 -0.114761" rpy="0 0 0"/>
-      <geometry>
-        <mesh filename="file://$(find mycobot_description)/meshes/link1.stl" scale="0.001 0.001 0.001"/>
-      </geometry>
-    </collision>
-  </link>
-  <link name="link2">
-    <inertial>
-      <origin xyz="0.036906585755672516 -3.4711337715265245e-07 0.06799995568162967" rpy="0 0 0"/>
-      <mass value="5.91988968680626"/>
-      <inertia ixx="0.0188" iyy="0.019335" izz="0.004161" ixy="0.0" iyz="-0.0" ixz="0.0"/>
-    </inertial>
-    <visual>
-      <origin xyz="-0.045 -0.060072 -0.199761" rpy="0 0 0"/>
-      <geometry>
-        <mesh filename="file://$(find mycobot_description)/meshes/link2.stl" scale="0.001 0.001 0.001"/>
-      </geometry>
-      <material name="silver"/>
-    </visual>
-    <collision>
-      <origin xyz="-0.045 -0.060072 -0.199761" rpy="0 0 0"/>
-      <geometry>
-        <mesh filename="file://$(find mycobot_description)/meshes/link2.stl" scale="0.001 0.001 0.001"/>
-      </geometry>
-    </collision>
-  </link>
-  <link name="link3">
-    <inertial>
-      <origin xyz="-0.03502268825299208 3.0162871079368603e-05 0.04949994627901161" rpy="0 0 0"/>
-      <mass value="4.802107093668197"/>
-      <inertia ixx="0.01014" iyy="0.010584" izz="0.003386" ixy="0.0" iyz="-4e-06" ixz="0.0"/>
-    </inertial>
-    <visual>
-      <origin xyz="-0.045 -0.060072 -0.335761" rpy="0 0 0"/>
-      <geometry>
-        <mesh filename="file://$(find mycobot_description)/meshes/link3.stl" scale="0.001 0.001 0.001"/>
-      </geometry>
-      <material name="silver"/>
-    </visual>
-    <collision>
-      <origin xyz="-0.045 -0.060072 -0.335761" rpy="0 0 0"/>
-      <geometry>
-        <mesh filename="file://$(find mycobot_description)/meshes/link3.stl" scale="0.001 0.001 0.001"/>
-      </geometry>
-    </collision>
-  </link>
-  <link name="link4">
-    <inertial>
-      <origin xyz="0.034423872869192323 6.191592391645295e-06 0.010576061998245623" rpy="0 0 0"/>
-      <mass value="2.265107015236222"/>
-      <inertia ixx="0.001595" iyy="0.001803" izz="0.001595" ixy="-0.0" iyz="-0.0" ixz="-0.000324"/>
-    </inertial>
-    <visual>
-      <origin xyz="-0.045 -0.060133 -0.434761" rpy="0 0 0"/>
-      <geometry>
-        <mesh filename="file://$(find mycobot_description)/meshes/link4.stl" scale="0.001 0.001 0.001"/>
-      </geometry>
-      <material name="silver"/>
-    </visual>
-    <collision>
-      <origin xyz="-0.045 -0.060133 -0.434761" rpy="0 0 0"/>
-      <geometry>
-        <mesh filename="file://$(find mycobot_description)/meshes/link4.stl" scale="0.001 0.001 0.001"/>
-      </geometry>
-    </collision>
-  </link>
-  <link name="link5">
-    <inertial>
-      <origin xyz="5.551115123125783e-17 2.6368392026507315e-05 0.04211661683454615" rpy="0 0 0"/>
-      <mass value="3.029827579494103"/>
-      <inertia ixx="0.0025" iyy="0.002976" izz="0.002441" ixy="0.0" iyz="-0.0" ixz="0.0"/>
-    </inertial>
-    <visual>
-      <origin xyz="-0.09 -0.06016 -0.479761" rpy="0 0 0"/>
-      <geometry>
-        <mesh filename="file://$(find mycobot_description)/meshes/link5.stl" scale="0.001 0.001 0.001"/>
-      </geometry>
-      <material name="silver"/>
-    </visual>
-    <collision>
-      <origin xyz="-0.09 -0.06016 -0.479761" rpy="0 0 0"/>
-      <geometry>
-        <mesh filename="file://$(find mycobot_description)/meshes/link5.stl" scale="0.001 0.001 0.001"/>
-      </geometry>
-    </collision>
-  </link>
-  <link name="link6">
-    <inertial>
-      <origin xyz="0.010000000000000203 2.2737115904641891e-07 -8.116903615906779e-08" rpy="0 0 0"/>
-      <mass value="0.6042068071016569"/>
-      <inertia ixx="0.00037" iyy="0.000205" izz="0.000205" ixy="0.0" iyz="0.0" ixz="0.0"/>
-    </inertial>
-    <visual>
-      <origin xyz="-0.13 -0.060191 -0.529761" rpy="0 0 0"/>
-      <geometry>
-        <mesh filename="file://$(find mycobot_description)/meshes/link6.stl" scale="0.001 0.001 0.001"/>
-      </geometry>
-      <material name="silver"/>
-    </visual>
-    <collision>
-      <origin xyz="-0.13 -0.060191 -0.529761" rpy="0 0 0"/>
-      <geometry>
-        <mesh filename="file://$(find mycobot_description)/meshes/link6.stl" scale="0.001 0.001 0.001"/>
-      </geometry>
-    </collision>
-  </link>
-  <!-- joint -->
-  <joint name="joint2_to_joint1" type="revolute">
-    <origin xyz="0.0 0.060072 0.114761" rpy="0 0 0"/>
-    <parent link="base_link"/>
-    <child link="link1"/>
-    <axis xyz="-0.0 0.0 1.0"/>
-    <limit effort = "1000.0" lower = "-2.87" upper = "2.87" velocity = "0"/>
-  </joint>
-  <joint name="joint3_to_joint2" type="revolute">
-    <origin xyz="0.045 0.0 0.085" rpy="0 0 0"/>
-    <parent link="link1"/>
-    <child link="link2"/>
-    <axis xyz="1.0 0.0 0.0"/>
-    <limit effort = "1000.0" lower = "-2.87" upper = "2.87" velocity = "0"/>
-  </joint>
-  <joint name="joint4_to_joint3" type="revolute">
-    <origin xyz="0.0 0.0 0.136" rpy="0 0 0"/>
-    <parent link="link2"/>
-    <child link="link3"/>
-    <axis xyz="-1.0 0.0 -0.0"/>
-    <limit effort = "1000.0" lower = "-2.87" upper = "2.87" velocity = "0"/>
-  </joint>
-  <joint name="joint5_to_joint4" type="revolute">
-    <origin xyz="0.0 6.1e-05 0.099" rpy="0 0 0"/>
-    <parent link="link3"/>
-    <child link="link4"/>
-    <axis xyz="1.0 -0.0 0.0"/>
-    <limit effort = "1000.0" lower = "-2.87" upper = "2.87" velocity = "0"/>
-  </joint>
-  <joint name="joint6_to_joint5" type="revolute">
-    <origin xyz="0.045 2.7e-05 0.045" rpy="0 0 0"/>
-    <parent link="link4"/>
-    <child link="link5"/>
-    <axis xyz="-0.0 0.000616 1.0"/>
-    <limit effort = "1000.0" lower = "-2.87" upper = "2.87" velocity = "0"/>
-  </joint>
-  <joint name="joint6output_to_joint6" type="revolute">
-    <origin xyz="0.04 3.1e-05 0.05" rpy="0 0 0"/>
-    <parent link="link5"/>
-    <child link="link6"/>
-    <axis xyz="1.0 -0.0 0.0"/>
-    <limit effort = "1000.0" lower = "-2.87" upper = "2.87" velocity = "0"/>
-  </joint>
-<!-- gripper joints -->
+<link name="base_link">
+  <inertial>
+    <origin xyz="-1.3994637957346424e-08 0.046320428630226694 0.053625500753973876" rpy="0 0 0"/>
+    <mass value="12.899764355948896"/>
+    <inertia ixx="0.033823" iyy="0.028162" izz="0.035033" ixy="0.0" iyz="-0.000755" ixz="0.0"/>
+  </inertial>
+  <visual>
+    <origin xyz="0 0 0" rpy="0 0 0"/>
+    <geometry>
+      <mesh filename="file://$(find mycobot_description)/meshes/base_link.stl" scale="0.001 0.001 0.001"/>
+    </geometry>
+    <material name="silver"/>
+  </visual>
+  <collision>
+    <origin xyz="0 0 0" rpy="0 0 0"/>
+    <geometry>
+      <mesh filename="file://$(find mycobot_description)/meshes/base_link.stl" scale="0.001 0.001 0.001"/>
+    </geometry>
+  </collision>
+</link>
+<link name="link1">
+  <inertial>
+    <origin xyz="0.006896766224730391 -3.4711337724979696e-07 0.05549014255068621" rpy="0 0 0"/>
+    <mass value="3.4735206294395446"/>
+    <inertia ixx="0.004461" iyy="0.004757" izz="0.002424" ixy="0.0" iyz="-0.0" ixz="-0.000777"/>
+  </inertial>
+  <visual>
+    <origin xyz="0.0 -0.060072 -0.114761" rpy="0 0 0"/>
+    <geometry>
+      <mesh filename="file://$(find mycobot_description)/meshes/link1.stl" scale="0.001 0.001 0.001"/>
+    </geometry>
+    <material name="silver"/>
+  </visual>
+  <collision>
+    <origin xyz="0.0 -0.060072 -0.114761" rpy="0 0 0"/>
+    <geometry>
+      <mesh filename="file://$(find mycobot_description)/meshes/link1.stl" scale="0.001 0.001 0.001"/>
+    </geometry>
+  </collision>
+</link>
+<link name="link2">
+  <inertial>
+    <origin xyz="0.03690658575567238 -3.4711337713183577e-07 0.06799995568162978" rpy="0 0 0"/>
+    <mass value="5.91988968680626"/>
+    <inertia ixx="0.0188" iyy="0.019335" izz="0.004161" ixy="0.0" iyz="0.0" ixz="0.0"/>
+  </inertial>
+  <visual>
+    <origin xyz="-0.045 -0.060072 -0.199761" rpy="0 0 0"/>
+    <geometry>
+      <mesh filename="file://$(find mycobot_description)/meshes/link2.stl" scale="0.001 0.001 0.001"/>
+    </geometry>
+    <material name="silver"/>
+  </visual>
+  <collision>
+    <origin xyz="-0.045 -0.060072 -0.199761" rpy="0 0 0"/>
+    <geometry>
+      <mesh filename="file://$(find mycobot_description)/meshes/link2.stl" scale="0.001 0.001 0.001"/>
+    </geometry>
+  </collision>
+</link>
+<link name="link3">
+  <inertial>
+    <origin xyz="-0.03502268825299208 -3.4711337702081346e-07 0.049499955681629404" rpy="0 0 0"/>
+    <mass value="4.802107093668197"/>
+    <inertia ixx="0.01014" iyy="0.010584" izz="0.003386" ixy="0.0" iyz="-0.0" ixz="0.0"/>
+  </inertial>
+  <visual>
+    <origin xyz="-0.045 -0.060072 -0.335761" rpy="0 0 0"/>
+    <geometry>
+      <mesh filename="file://$(find mycobot_description)/meshes/link3.stl" scale="0.001 0.001 0.001"/>
+    </geometry>
+    <material name="silver"/>
+  </visual>
+  <collision>
+    <origin xyz="-0.045 -0.060072 -0.335761" rpy="0 0 0"/>
+    <geometry>
+      <mesh filename="file://$(find mycobot_description)/meshes/link3.stl" scale="0.001 0.001 0.001"/>
+    </geometry>
+  </collision>
+</link>
+<link name="link4">
+  <inertial>
+    <origin xyz="0.03442387286919234 -3.4711337690979116e-07 0.010576082812437049" rpy="0 0 0"/>
+    <mass value="2.265107015236222"/>
+    <inertia ixx="0.001595" iyy="0.001803" izz="0.001595" ixy="0.0" iyz="0.0" ixz="-0.000324"/>
+  </inertial>
+  <visual>
+    <origin xyz="-0.045 -0.060072 -0.434761" rpy="0 0 0"/>
+    <geometry>
+      <mesh filename="file://$(find mycobot_description)/meshes/link4.stl" scale="0.001 0.001 0.001"/>
+    </geometry>
+    <material name="silver"/>
+  </visual>
+  <collision>
+    <origin xyz="-0.045 -0.060072 -0.434761" rpy="0 0 0"/>
+    <geometry>
+      <mesh filename="file://$(find mycobot_description)/meshes/link4.stl" scale="0.001 0.001 0.001"/>
+    </geometry>
+  </collision>
+</link>
+<link name="link5">
+  <inertial>
+    <origin xyz="6.938893903907228e-17 -3.4711337680570775e-07 0.04211665218776295" rpy="0 0 0"/>
+    <mass value="3.029827579494103"/>
+    <inertia ixx="0.0025" iyy="0.002976" izz="0.002441" ixy="0.0" iyz="-0.0" ixz="-0.0"/>
+  </inertial>
+  <visual>
+    <origin xyz="-0.09 -0.060072 -0.479761" rpy="0 0 0"/>
+    <geometry>
+      <mesh filename="file://$(find mycobot_description)/meshes/link5.stl" scale="0.001 0.001 0.001"/>
+    </geometry>
+    <material name="silver"/>
+  </visual>
+  <collision>
+    <origin xyz="-0.09 -0.060072 -0.479761" rpy="0 0 0"/>
+    <geometry>
+      <mesh filename="file://$(find mycobot_description)/meshes/link5.stl" scale="0.001 0.001 0.001"/>
+    </geometry>
+  </collision>
+</link>
+<link name="link6">
+  <inertial>
+    <origin xyz="0.010000000000000092 -3.471133767779522e-07 -4.4318370751028624e-08" rpy="0 0 0"/>
+    <mass value="0.6042068071016569"/>
+    <inertia ixx="0.00037" iyy="0.000205" izz="0.000205" ixy="0.0" iyz="0.0" ixz="0.0"/>
+  </inertial>
+  <visual>
+    <origin xyz="-0.13 -0.060072 -0.529761" rpy="0 0 0"/>
+    <geometry>
+      <mesh filename="file://$(find mycobot_description)/meshes/link6.stl" scale="0.001 0.001 0.001"/>
+    </geometry>
+    <material name="silver"/>
+  </visual>
+  <collision>
+    <origin xyz="-0.13 -0.060072 -0.529761" rpy="0 0 0"/>
+    <geometry>
+      <mesh filename="file://$(find mycobot_description)/meshes/link6.stl" scale="0.001 0.001 0.001"/>
+    </geometry>
+  </collision>
+</link>
+<link name="gripper_left1">
+  <inertial>
+    <origin xyz="0.011053321311780717 -0.005254043045734549 0.00013658058489207647" rpy="0 0 0"/>
+    <mass value="0.09307370524691046"/>
+    <inertia ixx="1e-05" iyy="3.5e-05" izz="4.2e-05" ixy="-1.3e-05" iyz="0.0" ixz="0.0"/>
+  </inertial>
+  <visual>
+    <origin xyz="-0.261438 -0.008607 -0.536903" rpy="0 0 0"/>
+    <geometry>
+      <mesh filename="file://$(find mycobot_description)/meshes/gripper_left1.stl" scale="0.001 0.001 0.001"/>
+    </geometry>
+    <material name="silver"/>
+  </visual>
+  <collision>
+    <origin xyz="-0.261438 -0.008607 -0.536903" rpy="0 0 0"/>
+    <geometry>
+      <mesh filename="file://$(find mycobot_description)/meshes/gripper_left1.stl" scale="0.001 0.001 0.001"/>
+    </geometry>
+  </collision>
+</link>
+<link name="gripper_right1">
+  <inertial>
+    <origin xyz="0.011064486332764245 0.00525722808018074 0.003559949036713861" rpy="0 0 0"/>
+    <mass value="0.0929857868716481"/>
+    <inertia ixx="1e-05" iyy="3.5e-05" izz="4.2e-05" ixy="1.3e-05" iyz="0.0" ixz="-0.0"/>
+  </inertial>
+  <visual>
+    <origin xyz="-0.261438 -0.111297 -0.533501" rpy="0 0 0"/>
+    <geometry>
+      <mesh filename="file://$(find mycobot_description)/meshes/gripper_right1.stl" scale="0.001 0.001 0.001"/>
+    </geometry>
+    <material name="silver"/>
+  </visual>
+  <collision>
+    <origin xyz="-0.261438 -0.111297 -0.533501" rpy="0 0 0"/>
+    <geometry>
+      <mesh filename="file://$(find mycobot_description)/meshes/gripper_right1.stl" scale="0.001 0.001 0.001"/>
+    </geometry>
+  </collision>
+</link>
+<link name="gripper_left3">
+  <inertial>
+    <origin xyz="0.01599044289886639 -0.012967874127836797 0.003475371537171479" rpy="0 0 0"/>
+    <mass value="0.09059526730883062"/>
+    <inertia ixx="1.8e-05" iyy="3.3e-05" izz="5e-05" ixy="1.8e-05" iyz="0.0" ixz="-0.0"/>
+  </inertial>
+  <visual>
+    <origin xyz="-0.21039 -0.041612 -0.533403" rpy="0 0 0"/>
+    <geometry>
+      <mesh filename="file://$(find mycobot_description)/meshes/gripper_left3.stl" scale="0.001 0.001 0.001"/>
+    </geometry>
+    <material name="silver"/>
+  </visual>
+  <collision>
+    <origin xyz="-0.21039 -0.041612 -0.533403" rpy="0 0 0"/>
+    <geometry>
+      <mesh filename="file://$(find mycobot_description)/meshes/gripper_left3.stl" scale="0.001 0.001 0.001"/>
+    </geometry>
+  </collision>
+</link>
+<link name="gripper_right3">
+  <inertial>
+    <origin xyz="0.015989588845322006 0.012966613242614375 0.0035542257609944006" rpy="0 0 0"/>
+    <mass value="0.09058559783383588"/>
+    <inertia ixx="1.8e-05" iyy="3.3e-05" izz="5e-05" ixy="-1.8e-05" iyz="-0.0" ixz="-0.0"/>
+  </inertial>
+  <visual>
+    <origin xyz="-0.21039 -0.078292 -0.533403" rpy="0 0 0"/>
+    <geometry>
+      <mesh filename="file://$(find mycobot_description)/meshes/gripper_right3.stl" scale="0.001 0.001 0.001"/>
+    </geometry>
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
File: src/mycobot_moveit/config/mycobot.ros2_control.xacro (robot description, xacro)
@@ -1,5 +1,5 @@
 <?xml version="1.0"?>
 <robot xmlns:xacro="http://www.ros.org/wiki/xacro">
-    <xacro:macro name="mycobot320_ros2_control" params="name initial_positions_file">
+    <xacro:macro name="mycobot_ros2_control" params="name initial_positions_file">
         <xacro:property name="initial_positions" value="${xacro.load_yaml(initial_positions_file)['initial_positions']}"/>
         <ros2_control name="${name}" type="system">
@@ -50,4 +50,11 @@
                 <state_interface name="velocity"/>
             </joint>
+            <joint name="gripper_controller">
+                <command_interface name="position"/>
+                <state_interface name="position">
+                  <param name="initial_value">${initial_positions['gripper_controller']}</param>
+                </state_interface>
+                <state_interface name="velocity"/>
+            </joint>
         </ros2_control>
     </xacro:macro>

Commit message: RohWS success

File: src/mycobot_description/urdf/mycobot.xacro (robot description, xacro)
@@ -338,5 +338,5 @@
   <child link="gripper_right1"/>
   <axis xyz="-0.0 -0.0 -1.0"/>
-  <limit upper="0.698132" lower="0.0" effort="100" velocity="100"/>
+  <limit upper="0.0" lower="-0.698132" effort="100" velocity="100"/>
   <mimic joint="gripper_controller" multiplier="-1" offset="0"/>
 </joint>

Commit message: success gripper, wow!

File: src/mycobot_description/urdf/mycobot.xacro (robot description, xacro)
@@ -327,12 +327,12 @@
 </joint>
 <joint name="gripper_controller" type="revolute">
-  <origin xyz="0.06039 0.01822 0.003642" rpy="0 0 0"/>
+  <origin xyz="0.06039 0.01822 0.003642" rpy="0 0 -0.42"/>
   <parent link="gripper_base"/>
   <child link="gripper_right3"/>
   <axis xyz="0.0 -0.0 -1.0"/>
-  <limit upper="0.698132" lower="0.0" effort="100" velocity="100"/>
+  <limit upper="0.3" lower="-0.7" effort="100" velocity="100"/>
 </joint>
 <joint name="gripper_right3_to_gripper_right1" type="revolute">
-  <origin xyz="0.051048 0.033005 9.8e-05" rpy="0 0 0"/>
+  <origin xyz="0.051048 0.033005 9.8e-05" rpy="0 0 0.42"/>
   <parent link="gripper_right3"/>
   <child link="gripper_right1"/>
@@ -350,5 +350,5 @@
 </joint> -->
 <joint name="gripper_left3_to_gripper_left1" type="revolute">
-  <origin xyz="0.051048 -0.033005 0.0035" rpy="0 0 0"/>
+  <origin xyz="0.051048 -0.033005 0.0035" rpy="0 0 -0.42"/>
   <parent link="gripper_left3"/>
   <child link="gripper_left1"/>
@@ -358,5 +358,5 @@
 </joint>
 <joint name="gripper_base_to_gripper_left3" type="revolute">
-  <origin xyz="0.06039 -0.01846 0.003642" rpy="0 0 0"/>
+  <origin xyz="0.06039 -0.01846 0.003642" rpy="0 0 0.42"/>
   <parent link="gripper_base"/>
   <child link="gripper_left3"/>

File: src/mycobot_moveit/config/mycobot.ros2_control.xacro (robot description, xacro)
@@ -13,5 +13,7 @@
                   <param name="initial_value">${initial_positions['joint2_to_joint1']}</param>
                 </state_interface>
-                <state_interface name="velocity"/>
+                <state_interface name="velocity">
+                  <param name="initial_value">0.0</param>
+                </state_interface>
             </joint>
             <joint name="joint3_to_joint2">
@@ -20,5 +22,7 @@
                   <param name="initial_value">${initial_positions['joint3_to_joint2']}</param>
                 </state_interface>
-                <state_interface name="velocity"/>
+                <state_interface name="velocity">
+                  <param name="initial_value">0.0</param>
+                </state_interface>
             </joint>
             <joint name="joint4_to_joint3">
@@ -27,5 +31,7 @@
                   <param name="initial_value">${initial_positions['joint4_to_joint3']}</param>
                 </state_interface>
-                <state_interface name="velocity"/>
+                <state_interface name="velocity">
+                  <param name="initial_value">0.0</param>
+                </state_interface>
             </joint>
             <joint name="joint5_to_joint4">
@@ -34,5 +40,7 @@
                   <param name="initial_value">${initial_positions['joint5_to_joint4']}</param>
                 </state_interface>
-                <state_interface name="velocity"/>
+                <state_interface name="velocity">
+                  <param name="initial_value">0.0</param>
+                </state_interface>
             </joint>
             <joint name="joint6_to_joint5">
@@ -41,5 +49,7 @@
                   <param name="initial_value">${initial_positions['joint6_to_joint5']}</param>
                 </state_interface>
-                <state_interface name="velocity"/>
+                <state_interface name="velocity">
+                  <param name="initial_value">0.0</param>
+                </state_interface>
             </joint>
             <joint name="joint6output_to_joint6">
@@ -48,5 +58,7 @@
                   <param name="initial_value">${initial_positions['joint6output_to_joint6']}</param>
                 </state_interface>
-                <state_interface name="velocity"/>
+                <state_interface name="velocity">
+                  <param name="initial_value">0.0</param>
+                </state_interface>
             </joint>
             <joint name="gripper_controller">
@@ -55,5 +67,7 @@
                   <param name="initial_value">${initial_positions['gripper_controller']}</param>
                 </state_interface>
-                <state_interface name="velocity"/>
+                <state_interface name="velocity">
+                  <param name="initial_value">0.0</param>
+                </state_interface>
             </joint>
         </ros2_control>

File: src/mycobot_moveit/config/mycobot.srdf.xacro (robot description, xacro)
@@ -33,12 +33,15 @@
     <group_state name="ready" group="mycobot_arm">
         <joint name="joint2_to_joint1" value="0"/>
-        <joint name="joint3_to_joint2" value="-0.5"/>
-        <joint name="joint4_to_joint3" value="0.2"/>
-        <joint name="joint5_to_joint4" value="-0.85"/>
-        <joint name="joint6_to_joint5" value="1.6"/>
+        <joint name="joint3_to_joint2" value="-0.3"/>
+        <joint name="joint4_to_joint3" value="0"/>
+        <joint name="joint5_to_joint4" value="-1.2"/>
+        <joint name="joint6_to_joint5" value="1.55"/>
         <joint name="joint6output_to_joint6" value="0"/>
     </group_state>
     <group_state name="open" group="gripper_group">
-        <joint name="gripper_controller" value="0"/>
+        <joint name="gripper_controller" value="-0.7"/>
+    </group_state>
+    <group_state name="close" group="gripper_group">
+        <joint name="gripper_controller" value="0.3"/>
     </group_state>
     <!--END EFFECTOR: Purpose: Represent information about an end effector.-->
